File: DeXIC/DeXIC.kicad_sch (KiCad schematic)
At the start: 0 parts

Commit message: first
Parts:
- added U1: CH32V003FxPx, Package_SO:TSSOP-20_4.4x6.5mm_P0.65mm, symbol MCU_WCH_RiscV:CH32V003FxPx

Commit message: Next
Parts:
- added BT1, BT2, BT3: Battery_Cell, symbol Device:Battery_Cell
- added C1, C2, C3, C4, C5, C6: 0.1uF, symbol Device:C
- added D1, D3, D9: Strike, symbol Device:LED
- added D10, D2, D4: Pass, symbol Device:LED
- added D5: Blue, symbol Device:LED
- added D6: White, symbol Device:LED
- added D7: Yellow, symbol Device:LED
- added D8: Red, symbol Device:LED
- added J1, J10, J4, J6, J8, J9: Conn_01x01_Socket, symbol Connector:Conn_01x01_Socket
- added J11, J12, J13, J2, J5, J7: ~, symbol Connector:Conn_01x01_Socket
- added J14, J21, J22: USART, symbol Connector:Conn_01x05_Pin
- added J28, J3, J30: Prog, symbol Connector:Conn_01x03_Pin
- added R1, R10, R11, R12, R13, R14, R15, R16, R17, R18, R19, R2, R20, R21, R3, R4, R5, R6, R7, R8, R9: 10k, symbol Device:R
- added SW1, SW2, SW3, SW4, SW5, SW6, SW7, SW8: SW_Push, symbol Switch:SW_Push
- added U2, U3: CH32V003FxPx, Package_SO:TSSOP-20_4.4x6.5mm_P0.65mm, symbol MCU_WCH_RiscV:CH32V003FxPx
Connections:
- net USART1_CK_0: now reaches U1.1 (PD4)
- net USART1_CK_0: now also J14.2 (Pin_2)
- net IO2_0: now reaches U1.10 (PC0)
- net IO2_0: now also J7.1 (Pin_1), R3.2
- net IO3_0: now reaches U1.11 (PC1)
- net IO3_0: now also J11.1 (Pin_1), R4.2
- net USART1_RTS_0: now reaches U1.12 (PC2)
- net USART1_RTS_0: now also J14.5 (Pin_5)
- net IO4_0: now reaches U1.13 (PC3)
- net IO4_0: now also J12.1 (Pin_1), R5.2
- net IO5_0: now reaches U1.14 (PC4)
- net IO5_0: now also J13.1 (Pin_1), R6.2
- net GND_0: now reaches U1.15 (PC5)
- net GND_0: now also U1.7 (VSS), BT1.2 (-), C1.2, C2.2, D1.1 (K), D2.1 (K), J1.1 (Pin_1), J10.1 (Pin_1), J3.3 (Pin_3), J4.1 (Pin_1), J6.1 (Pin_1), J8.1 (Pin_1), J9.1 (Pin_1), SW1.1
- net IO6_0: now reaches U1.16 (PC6)
- net IO6_0: now also R7.1
- net IO7_0: now reaches U1.17 (PC7)
- net IO7_0: now also R8.1
- net SWDIO_0: now reaches U1.18 (PD1)
- net SWDIO_0: now also J3.2 (Pin_2)
- net IO1_0: now reaches U1.19 (PD2)
- net IO1_0: now also J5.1 (Pin_1), R2.2
- net USART1_TX_0: now reaches U1.2 (PD5)
- net USART1_TX_0: now also J14.3 (Pin_3)
- net USART1_CTS_0: now reaches U1.20 (PD3)
- net USART1_CTS_0: now also J14.1 (Pin_1)
- net USART1_RX_0: now reaches U1.3 (PD6)
- net USART1_RX_0: now also J14.4 (Pin_4)
- net RST_0: now reaches U1.4 (PD7)
- net RST_0: now also C1.1, SW1.2
- net IO0_0: now reaches U1.8 (PD0)
- net IO0_0: now also J2.1 (Pin_1), R1.2
- net VDD_0: now reaches U1.9 (VDD)
- net VDD_0: now also BT1.1 (+), C2.1, J3.1 (Pin_1), R1.1, R2.1, R3.1, R4.1, R5.1, R6.1
- new net: D6.2 (A), R13.2
- new net: D4.2 (A), R10.2
- new net: D2.2 (A), R8.2
- new net: D3.2 (A), R9.2
- new net: D1.2 (A), R7.2
- new net: D10.2 (A), R17.2
- new net: D8.2 (A), R15.2
- new net: D9.2 (A), R16.2
- new net: D7.2 (A), R14.2
- new net: D5.2 (A), R12.2
- new net GND_1: BT2.2 (-), C3.2, C4.2, D3.1 (K), D4.1 (K), D5.1 (K), D6.1 (K), D7.1 (K), D8.1 (K), J28.3 (Pin_3), SW2.1, SW3.1, U2.15 (PC5), U2.7 (VSS)
- new net GND_2: BT3.2 (-), C5.2, C6.2, D10.1 (K), D9.1 (K), J30.3 (Pin_3), SW4.1, SW5.1, SW6.1, SW7.1, SW8.1, U3.15 (PC5), U3.7 (VSS)
- new net IO0_1: R11.2, SW3.2, U2.8 (PD0)
- new net IO0_2: R18.2, SW5.2, U3.8 (PD0)
- new net IO1_1: R12.1, U2.19 (PD2)
- new net IO1_2: R19.2, SW6.2, U3.19 (PD2)
- new net IO2_1: R13.1, U2.10 (PC0)
- new net IO2_2: R20.2, SW7.2, U3.10 (PC0)
- new net IO3_1: R14.1, U2.11 (PC1)
- new net IO3_2: R21.2, SW8.2, U3.11 (PC1)
- new net IO4_1: R15.1, U2.13 (PC3)
- new net IO4_2: U3.13 (PC3)
- new net IO5_1: U2.14 (PC4)
- new net IO5_2: U3.14 (PC4)
- new net IO6_1: R9.1, U2.16 (PC6)
- new net IO6_2: R16.1, U3.16 (PC6)
- new net IO7_1: R10.1, U2.17 (PC7)
- new net IO7_2: R17.1, U3.17 (PC7)
- new net RST_1: C3.1, SW2.2, U2.4 (PD7)
- new net RST_2: C5.1, SW4.2, U3.4 (PD7)
- new net SWDIO_1: J28.2 (Pin_2), U2.18 (PD1)
- new net SWDIO_2: J30.2 (Pin_2), U3.18 (PD1)
- new net USART1_CK_1: J21.2 (Pin_2), U2.1 (PD4)
- new net USART1_CK_2: J22.2 (Pin_2), U3.1 (PD4)
- new net USART1_CTS_1: J21.1 (Pin_1), U2.20 (PD3)
- new net USART1_CTS_2: J22.1 (Pin_1), U3.20 (PD3)
- new net USART1_RTS_1: J21.5 (Pin_5), U2.12 (PC2)
- new net USART1_RTS_2: J22.5 (Pin_5), U3.12 (PC2)
- new net USART1_RX_1: J21.4 (Pin_4), U2.3 (PD6)
- new net USART1_RX_2: J22.4 (Pin_4), U3.3 (PD6)
- new net USART1_TX_1: J21.3 (Pin_3), U2.2 (PD5)
- new net USART1_TX_2: J22.3 (Pin_3), U3.2 (PD5)
- new net VDD_1: BT2.1 (+), C4.1, J28.1 (Pin_1), R11.1, U2.9 (VDD)
- new net VDD_2: BT3.1 (+), C6.1, J30.1 (Pin_1), R18.1, R19.1, R20.1, R21.1, U3.9 (VDD)
- no-connect marks 0 -> 6
Other:
- note added: "Wire Module"

Commit message: Blashhh
Parts:
- added BT4: Battery_Cell, symbol Device:Battery_Cell
- added C7, C8: 0.1uF, symbol Device:C
- added D12, D13, D14, D16, D17, D18: D, symbol Device:D
- added J15: USART, symbol Connector:Conn_01x05_Pin
- added J16: Prog, symbol Connector:Conn_01x03_Pin
- added R22, R23, R24, R25: 10k, symbol Device:R
- added SW10, SW11, SW12, SW13, SW9: SW_Push, symbol Switch:SW_Push
- added U4: CH32V003FxPx, Package_SO:TSSOP-20_4.4x6.5mm_P0.65mm, symbol MCU_WCH_RiscV:CH32V003FxPx
Connections:
- net VDD_1: now also U4.9 (VDD)
- new net GND_3: BT4.2 (-), C7.2, C8.2, J16.3 (Pin_3), SW10.1, SW11.1, SW12.1, SW13.1, SW9.1, U4.15 (PC5), U4.7 (VSS)
- new net IO0_3: R22.2, SW10.2, U4.8 (PD0)
- new net IO1_3: R23.2, SW11.2, U4.19 (PD2)
- new net IO2_3: R24.2, SW12.2, U4.10 (PC0)
- new net IO3_3: R25.2, SW13.2, U4.11 (PC1)
- new net IO4_3: U4.13 (PC3)
- new net IO5_3: D12.2 (A), D13.2 (A), D14.1 (K), D17.1 (K), U4.14 (PC4)
- new net IO6_3: D12.1 (K), D14.2 (A), D16.2 (A), D18.1 (K), U4.16 (PC6)
- new net IO7_3: D13.1 (K), D16.1 (K), D17.2 (A), D18.2 (A), U4.17 (PC7)
- new net RST_3: C7.1, SW9.2, U4.4 (PD7)
- new net SWDIO_3: J16.2 (Pin_2), U4.18 (PD1)
- new net USART1_CK_3: J15.2 (Pin_2), U4.1 (PD4)
- new net USART1_CTS_3: J15.1 (Pin_1), U4.20 (PD3)
- new net USART1_RTS_3: J15.5 (Pin_5), U4.12 (PC2)
- new net USART1_RX_3: J15.4 (Pin_4), U4.3 (PD6)
- new net USART1_TX_3: J15.3 (Pin_3), U4.2 (PD5)
- new net VDD_3: BT4.1 (+), C8.1, J16.1 (Pin_1), R22.1, R23.1, R24.1, R25.1
- no-connect marks 6 -> 8
Other:
- note added: "Button"
- note added: "Keypad"
- note added: "Simon Says"
- moved on the sheet: BT1, BT2, BT3, C1, C2, C3, C4, C5, C6, D1, D10, D2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

Commit message: pcb
Parts:
- added BT5: Battery_Cell, Battery:BatteryHolder_Keystone_1042_1x18650, symbol Device:Battery_Cell
- added C10, C9: 0.1uF, Capacitor_THT:CP_Radial_D5.0mm_P2.00mm, symbol Device:C
- added D11: Strike, LED_THT:LED_D3.0mm, symbol Device:LED
- added D15: Pass, LED_THT:LED_D3.0mm_Clear, symbol Device:LED
- added J17: USART, Connector_PinHeader_2.54mm:PinHeader_1x05_P2.54mm_Vertical, symbol Connector:Conn_01x05_Pin
- added J18: Prog, Connector_PinHeader_2.54mm:PinHeader_1x03_P2.54mm_Vertical, symbol Connector:Conn_01x03_Pin
- added J19: 7 Segmentos, Connector_PinHeader_2.54mm:PinHeader_1x04_P2.54mm_Vertical, symbol Connector:Conn_01x04_Pin
- added R26, R27: 10k, Resistor_THT:R_Axial_DIN0204_L3.6mm_D1.6mm_P7.62mm_Horizontal, symbol Device:R
- added SW14: SW_Push, Button_Switch_THT:SW_PUSH-12mm_Wuerth-430476085716, symbol Switch:SW_Push
- added U5: CH32V003FxPx, Package_SO:TSSOP-20_4.4x6.5mm_P0.65mm, symbol MCU_WCH_RiscV:CH32V003FxPx
- BT1, BT2, BT3, BT4: footprint (none) -> Connector_PinHeader_2.54mm:PinHeader_2x01_P2.54mm_Vertical
- C1, C2, C3, C4, C5, C6, C7, C8: footprint (none) -> Capacitor_THT:CP_Radial_D5.0mm_P2.00mm
- D1, D3, D8, D9: footprint (none) -> LED_THT:LED_D3.0mm
- D10, D12, D13, D14, D16, D17, D18, D2, D4, D5, D6, D7: footprint (none) -> LED_THT:LED_D3.0mm_Clear
- J1, J10, J11, J12, J13, J2, J4, J5, J6, J7, J8, J9: footprint (none) -> Connector_PinHeader_2.54mm:PinHeader_1x01_P2.54mm_Vertical
- J14, J15, J21, J22: footprint (none) -> Connector_PinHeader_2.54mm:PinHeader_1x05_P2.54mm_Vertical
- J16, J28, J3, J30: footprint (none) -> Connector_PinHeader_2.54mm:PinHeader_1x03_P2.54mm_Vertical
- R1, R10, R11, R12, R13, R14, R15, R16, R17, R18, R19, R2, R20, R21, R22, R23, R24, R25, R3, R4, R5, R6, R7, R8, R9: footprint (none) -> Resistor_THT:R_Axial_DIN0204_L3.6mm_D1.6mm_P7.62mm_Horizontal
- SW1, SW10, SW11, SW12, SW13, SW2, SW3, SW4, SW5, SW6, SW7, SW8, SW9: footprint (none) -> Button_Switch_THT:SW_PUSH-12mm_Wuerth-430476085716
Connections:
- net VDD_1: no longer U4.9 (VDD)
- net VDD_3: now also U4.9 (VDD)
- new net: D15.2 (A), R27.2
- new net: D11.2 (A), R26.2
- new net GND_4: BT5.2 (-), C10.2, C9.2, D11.1 (K), D15.1 (K), J18.3 (Pin_3), J19.3 (Pin_3), SW14.1, U5.15 (PC5), U5.7 (VSS)
- new net IO0_4: J19.2 (Pin_2), U5.8 (PD0)
- new net IO1_4: J19.1 (Pin_1), U5.19 (PD2)
- new net IO2_4: U5.10 (PC0)
- new net IO3_4: U5.11 (PC1)
- new net IO4_4: U5.13 (PC3)
- new net IO5_4: U5.14 (PC4)
- new net IO6_4: R26.1, U5.16 (PC6)
- new net IO7_4: R27.1, U5.17 (PC7)
- new net RST_4: C9.1, SW14.2, U5.4 (PD7)
- new net SWDIO_4: J18.2 (Pin_2), U5.18 (PD1)
- new net USART1_CK_4: J17.2 (Pin_2), U5.1 (PD4)
- new net USART1_CTS_4: J17.1 (Pin_1), U5.20 (PD3)
- new net USART1_RTS_4: J17.5 (Pin_5), U5.12 (PC2)
- new net USART1_RX_4: J17.4 (Pin_4), U5.3 (PD6)
- new net USART1_TX_4: J17.3 (Pin_3), U5.2 (PD5)
- new net VDD_4: BT5.1 (+), C10.1, J18.1 (Pin_1), J19.4 (Pin_4), U5.9 (VDD)
- no-connect marks 8 -> 10
Other:
- note added: "Brain"
