File: DeXIC/DeXIC.kicad_pcb (KiCad board)
At the start: 2 copper layers, 70 x 70 mm, 102 parts, among them J1 Conn_01x01_Socket, J10 Conn_01x01_Socket, J14 USART, J15 USART, J16 Prog, J17 USART, J18 Prog, J19 7 Segmentos, J21 USART, J22 USART, J28 Prog, J3 Prog, J30 Prog, J4 Conn_01x01_Socket, J6 Conn_01x01_Socket, J8 Conn_01x01_Socket, J9 Conn_01x01_Socket, SW1 SW_Push, SW10 SW_Push, SW11 SW_Push, SW12 SW_Push, SW13 SW_Push, SW14 SW_Push, SW2 SW_Push, SW3 SW_Push, SW4 SW_Push, SW5 SW_Push, SW6 SW_Push, SW7 SW_Push, SW8 SW_Push, SW9 SW_Push, U1 CH32V003FxPx, U2 CH32V003FxPx, U3 CH32V003FxPx, U4 CH32V003FxPx, U5 CH32V003FxPx

Commit message: Final
Parts:
- BT3, BT4, J15, J16, J21, J22, J28, J30, SW2, SW4, SW9: moved to B.Cu
- moved SW14 164.5 mm to (210.4, 152.9), turned to 90 degrees
- moved J17 140.5 mm to (208.4, 135.8), turned to 90 degrees
- moved J16 136.6 mm to (117.4, 45.0), turned to -90 degrees
- moved R23 134.3 mm to (107.4, 71.4), turned to -90 degrees
- moved C9 133.8 mm to (209.4, 131.2), turned to 90 degrees
- moved C10 133.7 mm to (215.9, 131.2), turned to 90 degrees
- moved C7 127.5 mm to (121.0, 52.3)
- moved C8 127.5 mm to (121.0, 58.9)
- moved D16 126.2 mm to (113.8, 78.8), turned to 90 degrees
- moved D17 126.1 mm to (114.4, 92.3), turned to 90 degrees
- moved J19 124.6 mm to (208.4, 124.6), turned to 90 degrees
- moved U4 122.4 mm to (135.4, 57.0)
- moved R24 122.3 mm to (117.8, 105.0)
- moved D11 119.0 mm to (208.8, 120.6), turned to 90 degrees
- moved D15 118.8 mm to (214.3, 120.6), turned to 90 degrees
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Routing:
- net /GND_3: track 0.00 -> 241.3 mm
- net /GND_2: track 0.00 -> 219.3 mm
- net /GND_1: track 0.00 -> 212.8 mm
- net /VDD_3: track 0.00 -> 188.2 mm, vias 0 -> 2
- net /VDD_2: track 0.00 -> 179.2 mm, vias 0 -> 1
- net /IO5_3: track 0.00 -> 150.8 mm, vias 0 -> 1
- net /IO7_3: track 0.00 -> 121.8 mm, vias 0 -> 2
- net /IO6_3: track 0.00 -> 121.4 mm, vias 0 -> 1
- net /IO3_3: track 0.00 -> 107.0 mm, vias 0 -> 1
- net /VDD_0: track 54.0 -> 153.0 mm
- net /IO0_3: track 0.00 -> 92.9 mm
- net /GND_0: track 61.1 -> 145.7 mm, vias 0 -> 1
- net /IO0_1: track 0.00 -> 83.9 mm, vias 0 -> 1
- net /SWDIO_0: track 0.00 -> 76.3 mm
- net /VDD_1: track 0.00 -> 74.9 mm
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Other:
- board size 70 x 70 mm -> 145.9 x 143.8 mm
- board text added: "Button Module"
- board text added: "Keypad Module"
- board text added: "Simon Says Module"
- board text added: "Wire Module"
